Commit message: update to match our robot

File: linorobot2_description/urdf/2wd_properties.urdf.xacro (robot description, xacro)
@@ -1,16 +1,16 @@
 <?xml version="1.0"?>
 <robot xmlns:xacro="http://ros.org/wiki/xacro">
-  <xacro:property name="base_length" value="0.24" />
-  <xacro:property name="base_width" value="0.275" />
-  <xacro:property name="base_height" value="0.003" />
-  <xacro:property name="base_mass" value="1" />
-  <xacro:property name="wheel_radius" value="0.045" />
-  <xacro:property name="wheel_width" value="0.01" />
+  <xacro:property name="base_length" value="0.14" />
+  <xacro:property name="base_width" value="0.08" />
+  <xacro:property name="base_height" value="0.06" />
+  <xacro:property name="base_mass" value="0.1" />
+  <xacro:property name="wheel_radius" value="0.02" />
+  <xacro:property name="wheel_width" value="0.006" />
   <xacro:property name="wheel_pos_x" value="0.0" />
-  <xacro:property name="wheel_pos_y" value="0.13" />
+  <xacro:property name="wheel_pos_y" value="0.04" />
   <xacro:property name="wheel_pos_z" value="-0.03" />
   <xacro:property name="wheel_mass" value=".1" />
   <xacro:property name="wheel_torque" value="20" />
-  <xacro:property name="front_caster_wheel" value="true" />
+  <xacro:property name="front_caster_wheel" value="false" />
   <xacro:property name="rear_caster_wheel" value="true" />
   <xacro:property name="laser_pose">

File: linorobot2_description/urdf/mech/base.urdf.xacro (robot description, xacro)
@@ -5,5 +5,5 @@
     <link name="base_link">
       <visual>
-        <origin xyz="0 0 0" rpy="0 0 0"/>
+        <origin xyz="-0.0235 0 0" rpy="0 0 0"/>
         <geometry>
           <box size="${length} ${width} ${height}"/>
@@ -15,5 +15,5 @@
       </visual>
       <collision>
-        <origin xyz="0 0 0" rpy="0 0 0"/>
+        <origin xyz="-0.0235 0 0" rpy="0 0 0"/>
         <geometry>
           <box size="${length} ${width} ${height}"/>
@@ -21,5 +21,5 @@
       </collision>
       <inertial>
-        <origin xyz="0 0 0" rpy="0 0 0"/>
+        <origin xyz="-0.0235 0 0" rpy="0 0 0"/>
         <mass value="${mass}"/>
         <inertia ixx="${(1/12) * mass * ((width  * width)  + (height * height))}" ixy="0.0" ixz="0.0"

File: linorobot2_description/urdf/mech/caster_wheel.urdf.xacro (robot description, xacro)
@@ -11,5 +11,5 @@
     <link name="${side}_caster_wheel_link">
       <visual>
-        <origin xyz="0 0 0" rpy="0 0 0"/>
+        <origin xyz="-0.03 0 0" rpy="0 0 0"/>
         <geometry>
           <sphere radius="${caster_wheel_radius}" />

File: linorobot2_description/urdf/robots/2wd.urdf.xacro (robot description, xacro)
@@ -6,6 +6,6 @@
   <xacro:include filename="$(find linorobot2_description)/urdf/mech/caster_wheel.urdf.xacro" />
   <xacro:include filename="$(find linorobot2_description)/urdf/sensors/imu.urdf.xacro" />
-  <xacro:include filename="$(find linorobot2_description)/urdf/sensors/generic_laser.urdf.xacro" />
-  <xacro:include filename="$(find linorobot2_description)/urdf/sensors/depth_sensor.urdf.xacro" />
+  <!-- <xacro:include filename="$(find linorobot2_description)/urdf/sensors/generic_laser.urdf.xacro" /> -->
+  <!-- <xacro:include filename="$(find linorobot2_description)/urdf/sensors/depth_sensor.urdf.xacro" /> -->
   <xacro:include filename="$(find linorobot2_description)/urdf/controllers/diff_drive.urdf.xacro" />
   <xacro:base
@@ -54,10 +54,10 @@
   </xacro:if>
   <xacro:imu/>
-  <xacro:generic_laser>
+  <!-- <xacro:generic_laser>
     <xacro:insert_block name="laser_pose" />
-  </xacro:generic_laser>
-  <xacro:depth_sensor>
+  </xacro:generic_laser> -->
+  <!-- <xacro:depth_sensor>
     <xacro:insert_block name="depth_sensor_pose" />
-  </xacro:depth_sensor>
+  </xacro:depth_sensor> -->
   <xacro:diff_drive_controller
     wheel_separation="${wheel_pos_y * 2}"
